File: ESS688_OPL3_SoundCard/ESS688_OPL3_SoundCard/ESS688_OPL3_SoundCard.kicad_sch (KiCad schematic)
At the start: 13 parts, among them J1 Bus_ISA_16bit, SW1 SW_DIP_x06, U1 ES688, U2 NE558, U3 YAC512, U4 YMF262-M, U5 74LS244, U6 74LS245, U7 TLV9104, U8 LP2992-5.0

Commit message: analog part 80% finished
Parts:
- removed C1: C, symbol Device:C
- removed JP2: SolderJumper_3_Bridged12, Package_SON:WSON-8-1EP_6x5mm_P1.27mm_EP3.4x4mm, symbol Jumper:SolderJumper_3_Bridged12
- added C10, C11, C12, C13, C14, C15, C16, C17, C18, C19, C20, C21, C22, C8, C9: 100n, symbol Device:C
- added C2, C3: 20p, symbol Device:C
- added C23, C7: 10u, symbol Device:C
- added C24: 33p, symbol Device:C
- added C25, C26: 2n7, symbol Device:C
- added C27, C4: 4n7, symbol Device:C
- added C28, C6: 20u, symbol Device:C
- added C29, C30, C34, C35: 470n, symbol Device:C
- added C31: 47n, symbol Device:C
- added C32, C33: 1n5, symbol Device:C
- added C5: 10n, symbol Device:C
- added FB1: FerriteBead_Small, symbol Device:FerriteBead_Small
- added JP3: EN_ISA_OSC, symbol Jumper:SolderJumper_2_Open
- added JP4: FMCLK_SRC, Package_SON:WSON-8-1EP_6x5mm_P1.27mm_EP3.4x4mm, symbol Jumper:SolderJumper_3_Bridged12
- added R1: 33R, symbol Device:R
- added R2, R3: 2k2, symbol Device:R
- added Y1: Crystal_GND2, symbol Device:Crystal_GND2
- JP1: value SolderJumper_3_Bridged12 -> 688_SCLK
Connections:
- net +12V: now also FB1.1; no longer U8.1 (VIN), U8.3 (ON/~{OFF})
- net +5V: now also JP1.1 (A), C10.1, C11.1, C12.1, C13.1, C14.1, C17.1, C18.1, C19.1, C20.1, C8.1, C9.1
- net +5VA: now also U7.4 (V+), C15.1, C16.1, C21.1, C22.1, C7.1
- net GND: now also JP1.3 (B), U1.38 (REFSEL), U7.11 (V-), C10.2, C11.2, C12.2, C13.2, C14.2, C15.2, C16.2, C17.2, C18.2, C19.2, C2.2, C20.2, C21.2, C22.2, C23.2, C24.2, C25.2, C26.2, C27.2, C28.2, C3.2, C31.2, C32.2, C33.2, C4.2, C5.2, C6.2, C7.2, C8.2, C9.2, Y1.2
- net at J1.30 (OSC): now also JP3.1 (A)
- net OPL3_CH1: now reaches U3.10 (CH1)
- net OPL3_CH1: now also U7.12 (+), C25.1
- net OPL3_CH2: now reaches U3.11 (CH2)
- net OPL3_CH2: now also U7.10 (+), C26.1
- net at U3.12 (SWIN): now also R1.1
- net at U3.13 (AOUT): now also U7.3 (+), C24.1
- net at U3.14 (MP): now also U7.6 (-), U7.7
- net at U3.16 (CV): now also U7.5 (+), C23.1
- net at U8.4 (BP): now also C5.1
- net at JP1.2 (C): now also U1.82 (SCLK)
- net MUSIC_L: now reaches U7.13 (-)
- net MUSIC_L: now also U7.14, R2.2
- net at U4.24 (CLK): now also JP4.2 (C)
- net at U7.1: now also U7.2 (-), R1.2
- net MUSIC_R: now reaches U7.8
- net MUSIC_R: now also U7.9 (-), R3.2
- net at U1.30 (FOUT_L): now also C32.1, C34.2
- net at U1.31 (FOUT_R): now also C33.1, C35.2
- net at U1.32 (MUSIC_L): now also C29.1
- net at U1.33 (MUSIC_R): now also C30.1
- net at U1.40 (CIN_L): now also C34.1
- net at U1.41 (CIN_R): now also C35.1
- net at U1.42 (VREF): now also C31.1
- net at U1.43 (CMR): now also C28.1
- net at U1.79 (XO): now also C3.1, JP4.1 (A), Y1.3
- net at U1.80 (Xi): now also C2.1, Y1.1
- net at U1.81 (EXTCLK): now also JP3.2 (B), JP4.3 (B)
- new net: C6.1, FB1.2, U8.1 (VIN), U8.3 (ON/~{OFF})
- new net: C30.2, C4.1, R3.1
- new net: C27.1, C29.2, R2.1
Other:
- note added: "Bypass Caps ES688"
- note added: "Bypass Caps LS244, LS245, NE558, YMF262"
- note added: "Bypass Caps YAC512, TLV9104"
- note added: "CLK ISA.OSC"
- note added: "CLK from 688_XO"
- note added: "Connect ISA.OSC"
- note added: "ISA.OSC on EXTCLK"
- note added: "XTAL on XI, XO"
- moved on the sheet: U7A, U7B, U7C, U7D, U7E, U8

Commit message: joystick port circuitry and connector
Parts:
- added C1: 100n, symbol Device:C
- added C36, C37, C38, C39, C40, C41, C42, C43: 10n, symbol Device:C
- added J2: DA15_Socket_MountingHoles, Package_TO_SOT_SMD:SOT-23-5, symbol Connector:DA15_Socket_MountingHoles
- added R10, R11, R12, R13, R14, R15, R4, R5, R6, R7, R8, R9: 2k2, symbol Device:R
Connections:
- net +5V: now also R10.1, R11.1, R12.1, R13.1, R14.1, R15.1, R8.1, R9.1
- net GND: now also C1.2, C36.2, C37.2, C38.2, C39.2, C40.2, C41.2, C42.2, C43.2
- net JoyA_B1: now reaches U5.2 (I0)
- net JoyA_B1: now also C40.1, J2.2, R12.2
- net JoyA_B2: now reaches U5.4 (I1)
- net JoyA_B2: now also C41.1, J2.7, R13.2
- net JoyB_B1: now reaches U5.6 (I2)
- net JoyB_B1: now also C42.1, J2.10 (P10), R14.2
- net JoyB_B2: now reaches U5.8 (I3)
- net JoyB_B2: now also C43.1, J2.14 (P14), R15.2
- net at U2.1 (OUT_A), U5.11 (I0): now also R8.2
- net at U2.8 (OUT_B), U5.13 (I1): now also R10.2
- net at U2.9 (OUT_C), U5.15 (I2): now also R11.2
- net at U2.16 (OUT_D), U5.17 (I3): now also R9.2
- net at U2.10 (TIMG_C): now also C38.1, R6.2
- net at U2.15 (TIMG_D): now also C39.1, R7.2
- net at U2.2 (TIMG_A): now also C36.1, R4.2
- net at U2.4 (V_CTRL): now also C1.1
- net at U2.7 (TIMG_B): now also C37.1, R5.2
- new net JoyA_X: J2.3, R4.1
- new net JoyA_Y: J2.6, R5.1
- new net JoyB_X: J2.11 (P111), R6.1
- new net JoyB_Y: J2.13 (P13), R7.1
Other:
- note added: "ISA.OSC to 688.EXTCLK"
- note added: "YMF262.CLK from 688.XO"
- note added: "YMF262.CLK from ISA.OSC"
- note removed: "CLK ISA.OSC"
- note removed: "CLK from 688_XO"
- note removed: "Connect ISA.OSC"
- note removed: "FMRSTB can be used for Joystick port!"
- note removed: "ISA.OSC on EXTCLK"
- moved on the sheet: C17, C18, C19, C20, C21, C22, C5, C6, C7, FB1, U2, U5A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

Commit message: Gameport, Wavetable Header add
Parts:
- added C44, C45: 470n, symbol Device:C
- added D1: LED, LED_SMD:LED_Cree-XHP50_3V_HighDensity, symbol Device:LED
- added FB2, FB3, FB4, FB5: FerriteBead_Small, symbol Device:FerriteBead_Small
- added J3: Wavetable Port, symbol Connector_Generic:Conn_02x13_Odd_Even
- added R16, R17, R18, R19: 2k2, symbol Device:R
- added SW2: SW_DIP_x01, symbol Switch:SW_DIP_x01
- J2: value DA15_Socket_MountingHoles -> Game Port
Connections:
- net +12V: now also FB4.1
- net +5V: now also FB2.1, FB3.1, R18.2, R19.1
- net GND: now also J2.4, J2.5, J2.SH (PAD), J3.1 (Pin_1), J3.11 (Pin_11), J3.15 (Pin_15), J3.17 (Pin_17), J3.19 (Pin_19), J3.21 (Pin_21), J3.23 (Pin_23), J3.25 (Pin_25), J3.3 (Pin_3), J3.5 (Pin_5), J3.7 (Pin_7), J3.9 (Pin_9), SW2.2
- net -12V: now reaches J1.7 (-12V)
- net -12V: now also FB5.1
- net at R1.1: now also U7.1, U7.2 (-); no longer U3.12 (SWIN)
- net at J2.1: now also J2.8, J2.9 (P9), FB2.2
- net at J2.12 (P12): now also R16.2
- net at J2.15 (P15): now also R17.2
- net at U1.85 (~{FMRSTB}), U2.13 (~{RESET}), U4.3 (~{IC}): now also J3.26 (Pin_26)
- net at C30.1, U1.33 (MUSIC_R): now also C44.2
- net at C29.1, U1.32 (MUSIC_L): now also C45.2
- net at U1.55 (GPI0): now also R19.2, SW2.1
- net at U1.56 (GPI1): now also J3.4 (Pin_4), R17.1
- net at U1.57 (GPO0): now also D1.1 (K)
- net at U1.58 (GPO1): now also R16.1
- new net: R1.2, U3.12 (SWIN)
- new net: FB3.2, J3.10 (Pin_10), J3.14 (Pin_14), J3.6 (Pin_6)
- new net: FB4.2, J3.18 (Pin_18)
- new net: C44.1, J3.20 (Pin_20)
- new net: FB5.2, J3.22 (Pin_22)
- new net: D1.2 (A), R18.1
- new net: C45.1, J3.24 (Pin_24)
- no-connect marks 62 -> 66
Other:
- moved on the sheet: J2, R1
